File: pee_cee_bee.kicad_sch (KiCad schematic)
At the start: 0 parts

Commit message: put down basic components
Parts:
- added D1, D2, D3, D4: WS2812B, LED_SMD:LED_WS2812B_PLCC4_5.0x5.0mm_P3.2mm, symbol LED:WS2812B
- added J1: Conn_01x02, symbol Connector_Generic:Conn_01x02
- added SW1: SW_SPDT, symbol Switch:SW_SPDT
- added U1: ESP32-C3_SUPERMINI_TH, ESP32-C3_SUPERMINI_TH:MODULE_ESP32-C3_SUPERMINI_TH, symbol ESP32-C3_SUPERMINI_TH:ESP32-C3_SUPERMINI_TH
Connections:
- new net: D1.1 (VDD), D2.1 (VDD), D3.1 (VDD), D4.1 (VDD)
- new net: D1.2 (DOUT), D2.4 (DIN)
- new net: D1.4 (DIN), U1.5 (GPIO5)
- new net: D2.2 (DOUT), D3.4 (DIN)
- new net: SW1.2 (B), U1.5V
- new net: D3.2 (DOUT), D4.4 (DIN)
- new net BATT+: J1.1 (Pin_1)
- new net GND: D1.3 (VSS), D2.3 (VSS), D3.3 (VSS), D4.3 (VSS), J1.2 (Pin_2)

Commit message: schematic done? add servo, flap, capacitor
Parts:
- added C1: C, symbol Device:C
- added J2: Conn_01x03, symbol Connector_Generic:Conn_01x03
- added SW2: SW_Push, symbol Switch:SW_Push
Connections:
- net BATT+: now also SW1.1 (A)
- net GND: now also U1.G (GND), C1.2, J2.1 (Pin_1), SW2.1
- net +5V: now reaches D1.1 (VDD), D2.1 (VDD), D3.1 (VDD), D4.1 (VDD)
- net +5V: now also SW1.2 (B), U1.5V, C1.1, J2.2 (Pin_2)
- net flap: now reaches U1.3 (GPIO3)
- net flap: now also SW2.2
- net at U1.4 (GPIO4): now also J2.3 (Pin_3)
- no-connect marks 0 -> 10
Other:
- note added: "battery"
- note added: "linear servo"

Commit message: add capacitor and resistors
Parts:
- added R1: R, symbol Device:R
Connections:
- net at D1.4 (DIN): now also R1.2; no longer U1.5 (GPIO5)
- new net: R1.1, U1.5 (GPIO5)
Changed lines of the file:
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@@
-	)
-	(junction
-		(at 134.62 72.39)
-		(diameter 0)
-		(color 0 0 0 0)
 	)
 	(junction
@@
 	(wire
 		(pts
-			(xy 184.15 73.66) (xy 173.99 73.66)
-		)
-		(stroke
-			(width 0)
-			(type default)
-		)
-	)
-	(wire
-		(pts
 			(xy 133.35 52.07) (xy 133.35 72.39)
 		)
@@
 	(wire
 		(pts
-			(xy 92.71 118.11) (xy 92.71 92.71)
+			(xy 92.71 118.11) (xy 92.71 110.49)
 		)
 		(stroke
@@
 	(wire
 		(pts
-			(xy 134.62 72.39) (xy 135.89 72.39)
-		)
-		(stroke
-			(width 0)
-			(type default)
-		)
-	)
-	(wire
-		(pts
 			(xy 162.56 118.11) (xy 173.99 118.11)
 		)
@@
 	(wire
 		(pts
-			(xy 173.99 90.17) (xy 134.62 90.17)
+			(xy 92.71 102.87) (xy 92.71 92.71)
 		)
 		(stroke
@@
 	(wire
 		(pts
-			(xy 173.99 73.66) (xy 173.99 90.17)
-		)
-		(stroke
-			(width 0)
-			(type default)
-		)
-	)
-	(wire
-		(pts
 			(xy 104.14 53.34) (xy 104.14 57.15)
 		)
@@
 	(wire
 		(pts
-			(xy 134.62 90.17) (xy 134.62 72.39)
-		)
-		(stroke
-			(width 0)
-			(type default)
-		)
-	)
-	(wire
-		(pts
-			(xy 133.35 72.39) (xy 134.62 72.39)
+			(xy 133.35 72.39) (xy 135.89 72.39)
 		)
 		(stroke
@@
 	)
 	(symbol
+		(lib_id "power:+5V")
+		(at 184.15 73.66 0)
+		(unit 1)
+		(exclude_from_sim no)
+		(in_bom yes)
+		(on_board yes)
+		(dnp no)
+		(fields_autoplaced yes)
+		(property "Reference" "#PWR012"
+			(at 184.15 77.47 0)
+			(effects
+				(font
+					(size 1.27 1.27)
+				)
+				(hide yes)
+			)
+		)
+		(property "Value" "+5V"
+			(at 184.15 68.58 0)
+			(effects
+				(font
+					(size 1.27 1.27)
+				)
+			)
+		)
+		(property "Footprint" ""
+			(at 184.15 73.66 0)
+			(effects
+				(font
+					(size 1.27 1.27)
+				)
+				(hide yes)
+			)
+		)
+		(property "Datasheet" ""
+			(at 184.15 73.66 0)
+			(effects
+				(font
+					(size 1.27 1.27)
+				)
+				(hide yes)
+			)
+		)
+		(property "Description" "Power symbol creates a global label with name \"+5V\""
+			(at 184.15 73.66 0)
+			(effects
+				(font
+					(size 1.27 1.27)
+				)
+				(hide yes)
+			)
+		)
+		(pin "1"
+		)
+		(instances
+			(project ""
+				(path "/31437cee-bf64-4f5c-a317-d133f6d05bdf"
+					(reference "#PWR012")
+					(unit 1)
+				)
+			)
+		)
+	)
+	(symbol
 		(lib_id "Device:C")
 		(at 184.15 77.47 0)
@@
 					(unit 1)
 				)
+			)
+		)
+	)
+	(symbol
+		(lib_id "Device:R")
+		(at 92.71 106.68 0)
+		(unit 1)
+		(exclude_from_sim no)
+		(in_bom yes)
+		(on_board yes)
+		(dnp no)
+		(fields_autoplaced yes)
+		(property "Reference" "R1"
+			(at 95.25 105.4099 0)
+			(effects
+				(font
+					(size 1.27 1.27)
+				)
+				(justify left)
+			)
+		)
+		(property "Value" "R"
+			(at 95.25 107.9499 0)
+			(effects
+				(font
+					(size 1.27 1.27)
+				)
+				(justify left)
+			)
+		)
+		(property "Footprint" ""
+			(at 90.932 106.68 90)
+			(effects
+				(font
+					(size 1.27 1.27)
+				)
+				(hide yes)
+			)
+		)
+		(property "Datasheet" "~"
+			(at 92.71 106.68 0)
+			(effects
+				(font
+					(size 1.27 1.27)
+				)
+				(hide yes)
+			)
+		)
+		(property "Description" "Resistor"
+			(at 92.71 106.68 0)
+			(effects
+				(font
+					(size 1.27 1.27)
+				)
+				(hide yes)
+			)
+		)
+		(pin "1"
+		)
+		(pin "2"
+		)
+		(instances
+			(project ""
+				(path "/31437cee-bf64-4f5c-a317-d133f6d05bdf"
+					(reference "R1")
+					(unit 1)
+				)
